File: Project/Group_11.sch (EAGLE design)
At the start: 29 parts, among them J1 POWER_JACKPTH_LOCK, U1 +12v

Commit message: Correzione schematico collegamenti MUX
Connections:
- removed net MUX_A0/1.3C: U$3.A0
- removed net MUX_A0/2.3C: U$2.P_1.7
- removed net MUX_A1/1.4C: U$3.A1
- removed net MUX_A1/2.3C: U$2.P_1.6
- removed net MUX_A2/1.4C: U$3.A2
- removed net MUX_A2/2.3C: U$2.P_1.5
- removed net MUX_OUT/1.4C: U$3.D
- removed net MUX_OUT/2.5C: U$2.P_1.4
- new net MUX_A0: U$2.P_1.7, U$3.A0
- new net MUX_A1: U$2.P_1.6, U$3.A1
- new net MUX_A2: U$2.P_1.5, U$3.A2
- new net MUX_OUT: U$2.P_1.4, U$3.D
Changed lines of the file:
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@@
-</segment>
-</net>
-<net name="MUX_A0/2.3C" class="0">
-<segment>
-<pinref part="U$2" gate="G$1" pin="P_1.7"/>
-<wire x1="114.3" y1="88.9" x2="114.3" y2="104.14" width="0.1524" layer="91"/>
-<label x="114.3" y="104.14" size="1.778" layer="95" rot="R90" xref="yes"/>
-</segment>
-</net>
-<net name="MUX_A1/2.3C" class="0">
-<segment>
-<pinref part="U$2" gate="G$1" pin="P_1.6"/>
-<wire x1="116.84" y1="88.9" x2="116.84" y2="104.14" width="0.1524" layer="91"/>
-<label x="116.84" y="104.14" size="1.778" layer="95" rot="R90" xref="yes"/>
-</segment>
-</net>
-<net name="MUX_A2/2.3C" class="0">
-<segment>
-<pinref part="U$2" gate="G$1" pin="P_1.5"/>
-<wire x1="119.38" y1="88.9" x2="119.38" y2="104.14" width="0.1524" layer="91"/>
-<label x="119.38" y="104.14" size="1.778" layer="95" rot="R90" xref="yes"/>
-</segment>
-</net>
-<net name="MUX_OUT/2.5C" class="0">
-<segment>
-<pinref part="U$2" gate="G$1" pin="P_1.4"/>
-<wire x1="121.92" y1="88.9" x2="121.92" y2="104.14" width="0.1524" layer="91"/>
-<label x="121.92" y="104.14" size="1.778" layer="95" rot="R90" xref="yes"/>
 </segment>
 </net>
@@
 </segment>
 </net>
-<net name="MUX_OUT/1.4C" class="0">
+<net name="MUX_OUT" class="0">
 <segment>
 <pinref part="U$3" gate="G$1" pin="D"/>
@@
 <label x="436.88" y="86.36" size="1.778" layer="95" xref="yes"/>
 </segment>
-</net>
-<net name="MUX_A0/1.3C" class="0">
+<segment>
+<pinref part="U$2" gate="G$1" pin="P_1.4"/>
+<wire x1="121.92" y1="88.9" x2="121.92" y2="104.14" width="0.1524" layer="91"/>
+<label x="121.92" y="104.14" size="1.778" layer="95" rot="R90" xref="yes"/>
+</segment>
+</net>
+<net name="MUX_A0" class="0">
 <segment>
 <pinref part="U$3" gate="G$1" pin="A0"/>
@@
 <label x="406.4" y="81.28" size="1.778" layer="95" rot="R180" xref="yes"/>
 </segment>
-</net>
-<net name="MUX_A1/1.4C" class="0">
+<segment>
+<pinref part="U$2" gate="G$1" pin="P_1.7"/>
+<wire x1="114.3" y1="88.9" x2="114.3" y2="104.14" width="0.1524" layer="91"/>
+<label x="114.3" y="104.14" size="1.778" layer="95" rot="R90" xref="yes"/>
+</segment>
+</net>
+<net name="MUX_A1" class="0">
 <segment>
 <pinref part="U$3" gate="G$1" pin="A1"/>
@@
 <label x="406.4" y="78.74" size="1.778" layer="95" rot="R180" xref="yes"/>
 </segment>
-</net>
-<net name="MUX_A2/1.4C" class="0">
+<segment>
+<pinref part="U$2" gate="G$1" pin="P_1.6"/>
+<wire x1="116.84" y1="88.9" x2="116.84" y2="104.14" width="0.1524" layer="91"/>
+<label x="116.84" y="104.14" size="1.778" layer="95" rot="R90" xref="yes"/>
+</segment>
+</net>
+<net name="MUX_A2" class="0">
 <segment>
 <pinref part="U$3" gate="G$1" pin="A2"/>
@@
 <label x="406.4" y="76.2" size="1.778" layer="95" rot="R180" xref="yes"/>
 </segment>
-</net>
+<segment>
+<pinref part="U$2" gate="G$1" pin="P_1.5"/>
+<wire x1="119.38" y1="88.9" x2="119.38" y2="104.14" width="0.1524" layer="91"/>
+<label x="119.38" y="104.14" size="1.778" layer="95" rot="R90" xref="yes"/>
+</segment>
+</net>
