File: Project/Group_11.brd (EAGLE design)
At the start: 29 parts, among them J1 POWER_JACKPTH_LOCK, U1 +12v

Commit message: Final version
Parts:
- moved J1 16.1 mm to (32.1, 45.6), turned to 180 degrees
- moved U2 1.37 mm to (40.6, 43.7)
- moved C1 1.27 mm to (25.1, 38.7)
- moved C3 0.38 mm to (38.1, 33.0)
- moved R10 0.38 mm to (12.3, 43.2)
Routing:
- net N$9: track 27.1 -> 36.0 mm
- net GND: track 14.3 -> 22.1 mm
- net MUX_A0: track 55.0 -> 53.8 mm
- net 5V: track 44.7 -> 43.7 mm
- net TEMP_OUT: track 42.7 -> 43.3 mm
